File: pcb/mini-remote/mini-remote.kicad_pcb (KiCad board)
At the start: 2 copper layers, 45.5 x 98 mm, 37 parts, among them J1 Conn_01x04, Q1 MMBT3906, SW1 SW_SPST, SW10 SW_SPST, SW11 SW_SPST, SW12 SW_SPST, SW13 SW_SPST, SW14 SW_SPST, SW15 SW_SPST, SW16 SW_SPST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

Commit message: Fix pcb error
Parts:
- removed the G*** at (147.5, 133.2)
Routing:
- net VCC: track 91.4 -> 103.1 mm, vias 2 -> 0

Commit message: PCB version 1
Parts:
- removed SW2, SW9: SW_SPST, Local:LL3301NF065QG
- added J2: Conn_01x02, Connector_PinHeader_2.54mm:PinHeader_1x02_P2.54mm_Vertical, B.Cu at (164.8, 87.8)
- added REF**: MountingHole_2.2mm_M2, MountingHole:MountingHole_2.2mm_M2, F.Cu at (147.5, 95.8)
- added SW19: SW_SPST, Local:LL3301NF065QG, F.Cu at (132.5, 143.0)
- added SW20: SW_SPST, Local:LL3301NF065QG, F.Cu at (147.5, 143.0)
- added SW21: SW_SPST, Local:LL3301NF065QG, F.Cu at (162.5, 143.0)
- R3: value 100 -> 1k; footprint Resistor_THT:R_Axial_DIN0207_L6.3mm_D2.5mm_P7.62mm_Horizontal -> Resistor_SMD:R_0805_2012Metric
- moved SW3 41.2 mm to (162.5, 54.5)
- moved J1 33.6 mm to (130.2, 92.8), turned to 0 degrees
- moved SW4 32.9 mm to (132.5, 68.0)
- moved SW6 22.1 mm to (162.5, 68.0)
- moved SW8 15.7 mm to (155.5, 89.0)
- moved SW7 15.4 mm to (140.0, 89.0)
- moved SW5 15.0 mm to (147.5, 68.0)
- moved SW10 13.5 mm to (132.5, 102.5)
- moved SW11 13.5 mm to (147.5, 102.5)
- moved SW12 13.5 mm to (162.5, 102.5)
- moved SW13 13.5 mm to (132.5, 116.0)
- moved SW14 13.5 mm to (147.5, 116.0)
- moved SW15 13.5 mm to (162.5, 116.0)
- moved SW16 13.5 mm to (132.5, 129.5)
- moved SW17 13.5 mm to (147.5, 129.5)
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- renumbered SW19 to SW22
Connections:
- net Net-(R3-Pad2) renamed /LED
- U1 pad 16: Net-(U1-Pad16) -> /ROW6
- U1 pad 5: Net-(U1-Pad5) -> /A2
- U1 pad 6: Net-(U1-Pad6) -> /A3
Routing:
- net /ROW6: track 0.00 -> 111.0 mm, vias 0 -> 1
- net /COL2: track 77.9 -> 185.1 mm
- net /COL0: track 126.1 -> 228.2 mm
- net /COL1: track 139.6 -> 198.5 mm
- net /ROW2: track 78.9 -> 21.6 mm
- net /ROW3: track 92.8 -> 49.0 mm
- net /ROW5: track 121.9 -> 78.2 mm
- net /ROW4: track 107.3 -> 63.6 mm
- net /ROW1: track 73.5 -> 33.9 mm
- net /A3: track 0.00 -> 35.6 mm
- net /A2: track 0.00 -> 33.3 mm
- net /ROW0: track 42.4 -> 60.6 mm
- net VCC: track 103.1 -> 110.9 mm
- net /SWIM: track 43.4 -> 37.4 mm
- net /LED: track 28.1 -> 33.8 mm, vias 1 -> 2
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Other:
- board text added: "A2"
- board text added: "A3"
- board text added: "version 1 - JLCJLCJLCJLC"
