File: pcb/mini-remote/mini-remote.sch (KiCad schematic (older format))
At the start: 31 parts, among them J1 Conn_01x04, Q1 MMBT3906, SW1 SW_SPST, SW10 SW_SPST, SW11 SW_SPST, SW12 SW_SPST, SW13 SW_SPST, SW14 SW_SPST, SW15 SW_SPST, SW16 SW_SPST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

Commit message: Fix pcb error
Parts:
- R3: value 100 -> 1k
Changed lines of the file:
@@
 P 5850 2700
 F 0 "R3" H 5920 2746 50  0000 L CNN
-F 1 "100" H 5920 2655 50  0000 L CNN
+F 1 "1k" H 5920 2655 50  0000 L CNN
 F 2 "Resistor_THT:R_Axial_DIN0207_L6.3mm_D2.5mm_P7.62mm_Horizontal" V 5780 2700 50  0001 C CNN
 F 3 "~" H 5850 2700 50  0001 C CNN

Commit message: PCB version 1
Parts:
- removed SW2, SW9: SW_SPST, Local:LL3301NF065QG, symbol Switch:SW_SPST
- added J2: Conn_01x02, Connector_PinHeader_2.54mm:PinHeader_1x02_P2.54mm_Vertical, symbol Connector_Generic:Conn_01x02
- added SW19, SW20, SW21: SW_SPST, Local:LL3301NF065QG, symbol Switch:SW_SPST
- renumbered SW19 to SW22
Connections:
- net COL0: now also SW19.1 (A)
- net COL1: now also SW20.1 (A)
- net COL2: now also SW21.1 (A)
- net ROW6: now reaches U1.16 (PB6)
- net ROW6: now also SW19.2 (B), SW20.2 (B), SW21.2 (B)
- net A2: now reaches U1.5 (PA2)
- net A2: now also J2.1 (Pin_1)
- net A3: now reaches U1.6 (PA3)
- net A3: now also J2.2 (Pin_2)
- net LED: now reaches R3.2, U1.9 (PD0)
- no-connect marks 6 -> 3
Other:
- moved on the sheet: BT1, C1, D2, R3, U1

Commit message: Fix wrong footprint in schematic
Parts:
- R3: footprint Resistor_THT:R_Axial_DIN0207_L6.3mm_D2.5mm_P7.62mm_Horizontal -> Resistor_SMD:R_0805_2012Metric
Changed lines of the file:
@@
 F 0 "R3" H 6320 2746 50  0000 L CNN
 F 1 "1k" H 6320 2655 50  0000 L CNN
-F 2 "Resistor_THT:R_Axial_DIN0207_L6.3mm_D2.5mm_P7.62mm_Horizontal" V 6180 2700 50  0001 C CNN
+F 2 "Resistor_SMD:R_0805_2012Metric" V 6180 2700 50  0001 C CNN
 F 3 "~" H 6250 2700 50  0001 C CNN
 	1    6250 2700
